Commit message: Added stomp planner, fixed world, tested pick and place

File: robotiq/robotiq_description/urdf/2f_85.ros2_control.xacro (robot description, xacro)
@@ -43,5 +43,5 @@
                 <command_interface name="position" />
                 <state_interface name="position">
-                    <param name="initial_value">0.6</param>
+                    <param name="initial_value">0.0</param>
                 </state_interface>
                 <state_interface name="velocity"/>

File: ur_simulation_gz/urdf/ur_gz.urdf.xacro (robot description, xacro)
@@ -87,4 +87,14 @@
     </plugin>
   </gazebo>
+  <gazebo reference="robotiq_85_left_finger_tip_link">
+  <sensor name='sensor_contact' type='contact'>
+    <contact>
+        <collision>robotiq_85_left_finger_tip_link_collision</collision>
+        <topic>/gripper_contact</topic>
+    </contact>
+      <always_on>1</always_on>
+      <update_rate>100</update_rate>
+    </sensor>
+  </gazebo>
   <!-- ros2 control instance -->
   <xacro:ur_ros2_control

Commit message: changed to effort controllers for gripper, tuned pid values, fixed gripper urdf

File: robotiq/robotiq_description/urdf/2f_85.ros2_control.xacro (robot description, xacro)
@@ -41,18 +41,17 @@
             <!-- With Gazebo or Hardware, they handle mimic joints, so we only need this command interface activated -->
             <joint name="${prefix}robotiq_85_left_knuckle_joint">
-                <command_interface name="position" />
-                <state_interface name="position">
-                    <param name="initial_value">0.0</param>
-                </state_interface>
+                <command_interface name="effort" />
+                <state_interface name="position"/>
                 <state_interface name="velocity"/>
+                <state_interface name="effort"/>
+            </joint>
+            <joint name="${prefix}robotiq_85_right_knuckle_joint">
+                <command_interface name="effort" />
+                <state_interface name="position"/>
+                <state_interface name="velocity"/>
+                <state_interface name="effort"/>
             </joint>
             <!-- When simulating we need to include the rest of the gripper joints -->
             <xacro:if value="${use_fake_hardware or sim_isaac or sim_gazebo}">
-                <joint name="${prefix}robotiq_85_right_knuckle_joint">
-                    <xacro:unless value="${sim_gazebo}">
-                        <state_interface name="position"/>
-                        <state_interface name="velocity"/>
-                    </xacro:unless>
-                </joint>
                 <joint name="${prefix}robotiq_85_left_inner_knuckle_joint">
                     <xacro:unless value="${sim_gazebo}">

File: robotiq/robotiq_description/urdf/robotiq_2f_85_macro.urdf.xacro (robot description, xacro)
@@ -160,51 +160,51 @@
                     <friction>
                     <ode>
-                        <mu1>100000.0</mu1>
-                        <mu2>100000.0</mu2>
+                        <mu1>10000</mu1>
+                        <mu2>10000</mu2>
                     </ode>
                     </friction>
                     <contact>
                     <ode>
-                        <kp>1e+5</kp>
-                        <kd>1</kd>
+                        <kp>10000</kp>
+                        <kd>0.1</kd>
+                        <soft_cfm>0</soft_cfm>
+                        <soft_erp>0.2</soft_erp>
+                        <minDepth>0.02</minDepth>
+                        <maxVel>0.5</maxVel>
+                    </ode>
+                    </contact>
+                </surface>
+            </collision>
+            <inertial>
+                <origin xyz="-0.01456706 -0.0008 0.01649701" rpy="0 0 0" />
+                <mass value="4.268588744e-02" />
+                <inertia ixx="1.048152e-05" iyy="1.197888e-05" izz="4.22784e-06" ixy="0.0" ixz="3.5232e-6" iyz="0.0" />
+            </inertial>
+        </link>
+        <link name="${prefix}robotiq_85_right_finger_tip_link">
+            <visual>
+                <geometry>
+                    <mesh filename="file://$(find robotiq_description)/meshes/visual/2f_85/right_finger_tip.dae" />
+                </geometry>
+            </visual>
+            <collision>
+                <geometry>
+                    <mesh filename="file://$(find robotiq_description)/meshes/collision/2f_85/right_finger_tip.stl" />
+                </geometry>
+                <surface>
+                    <friction>
+                    <ode>
+                        <mu1>10000</mu1>
+                        <mu2>10000</mu2>
+                    </ode>
+                    </friction>
+                    <contact>
+                    <ode>
+                        <kp>10000</kp>
+                        <kd>0.1</kd>
                         <soft_cfm>0</soft_cfm>
                         <soft_erp>0.2</soft_erp>
                         <minDepth>0.002</minDepth>
-                        <maxVel>0</maxVel>
-                    </ode>
-                    </contact>
-                </surface>
-            </collision>
-            <inertial>
-                <origin xyz="-0.01456706 -0.0008 0.01649701" rpy="0 0 0" />
-                <mass value="4.268588744e-02" />
-                <inertia ixx="1.048152e-05" iyy="1.197888e-05" izz="4.22784e-06" ixy="0.0" ixz="3.5232e-6" iyz="0.0" />
-            </inertial>
-        </link>
-        <link name="${prefix}robotiq_85_right_finger_tip_link">
-            <visual>
-                <geometry>
-                    <mesh filename="file://$(find robotiq_description)/meshes/visual/2f_85/right_finger_tip.dae" />
-                </geometry>
-            </visual>
-            <collision>
-                <geometry>
-                    <mesh filename="file://$(find robotiq_description)/meshes/collision/2f_85/right_finger_tip.stl" />
-                </geometry>
-                <surface>
-                    <friction>
-                    <ode>
-                        <mu1>100000.0</mu1>
-                        <mu2>100000.0</mu2>
-                    </ode>
-                    </friction>
-                    <contact>
-                    <ode>
-                        <kp>1e+5</kp>
-                        <kd>1</kd>
-                        <soft_cfm>0</soft_cfm>
-                        <soft_erp>0.2</soft_erp>
-                        <minDepth>0.002</minDepth>
-                        <maxVel>0</maxVel>
+                        <maxVel>0.5</maxVel>
                     </ode>
                     </contact>
@@ -227,5 +227,5 @@
             <axis xyz="0 -1 0" />
             <origin xyz="0.03060114 0.0 0.05490452" rpy="0 0 0" />
-            <limit lower="0.0" upper="0.8" velocity="0.5" effort="50" />
+            <limit lower="0.0" upper="0.8" velocity="1.0" effort="28" />
         </joint>
         <joint name="${prefix}robotiq_85_right_knuckle_joint" type="revolute">
@@ -234,6 +234,5 @@
             <axis xyz="0 -1 0" />
             <origin xyz="-0.03060114 0.0 0.05490452" rpy="0 0 0" />
-            <limit lower="-0.8" upper="0.0" velocity="0.5" effort="50" />
-            <mimic joint="${prefix}robotiq_85_left_knuckle_joint" multiplier="-1" />
+            <limit lower="-0.8" upper="0.0" velocity="1.0" effort="28" />
         </joint>
         <joint name="${prefix}robotiq_85_left_finger_joint" type="fixed">
@@ -275,4 +274,20 @@
             <mimic joint="${prefix}robotiq_85_left_knuckle_joint" />
         </joint>
+        <transmission name="robotiq_85_right_knuckle_joint_transmission">
+          <type>transmission_interface/SimpleTransmission</type>
+          <joint name="robotiq_85_right_knuckle_joint">
+            <hardwareInterface>EffortJointInterface</hardwareInterface>
+          </joint>
+          <actuator name="robotiq_85_right_knuckle_joint_actuator">
+          </actuator>
+        </transmission>
+        <transmission name="robotiq_85_leftknuckle_joint_transmission">
+          <type>transmission_interface/SimpleTransmission</type>
+          <joint name="robotiq_85_left_knuckle_joint">
+            <hardwareInterface>EffortJointInterface</hardwareInterface>
+          </joint>
+          <actuator name="robotiq_85_left_knuckle_joint_actuator">
+          </actuator>
+        </transmission>
     </xacro:macro>
 </robot>

File: ur5_moveit_config/config/ur.ros2_control.xacro (robot description, xacro)
@@ -10,50 +10,81 @@
             <joint name="shoulder_pan_joint">
                 <command_interface name="position"/>
+                <command_interface name="velocity"/>
+                <command_interface name="effort"/>
                 <state_interface name="position">
                   <param name="initial_value">${initial_positions['shoulder_pan_joint']}</param>
                 </state_interface>
                 <state_interface name="velocity"/>
+                <state_interface name="effort"/>
             </joint>
             <joint name="shoulder_lift_joint">
                 <command_interface name="position"/>
+                <command_interface name="velocity"/>
+                <command_interface name="effort"/>
                 <state_interface name="position">
                   <param name="initial_value">${initial_positions['shoulder_lift_joint']}</param>
                 </state_interface>
                 <state_interface name="velocity"/>
+                <state_interface name="effort"/>
             </joint>
             <joint name="elbow_joint">
                 <command_interface name="position"/>
+                <command_interface name="velocity"/>
+                <command_interface name="effort"/>
                 <state_interface name="position">
                   <param name="initial_value">${initial_positions['elbow_joint']}</param>
                 </state_interface>
                 <state_interface name="velocity"/>
+                <state_interface name="effort"/>
             </joint>
             <joint name="wrist_1_joint">
                 <command_interface name="position"/>
+                <command_interface name="velocity"/>
+                <command_interface name="effort"/>
                 <state_interface name="position">
                   <param name="initial_value">${initial_positions['wrist_1_joint']}</param>
                 </state_interface>
                 <state_interface name="velocity"/>
+                <state_interface name="effort"/>
             </joint>
             <joint name="wrist_2_joint">
                 <command_interface name="position"/>
+                <command_interface name="velocity"/>
+                <command_interface name="effort"/>
                 <state_interface name="position">
                   <param name="initial_value">${initial_positions['wrist_2_joint']}</param>
                 </state_interface>
                 <state_interface name="velocity"/>
+                <state_interface name="effort"/>
             </joint>
             <joint name="wrist_3_joint">
                 <command_interface name="position"/>
+                <command_interface name="velocity"/>
+                <command_interface name="effort"/>
                 <state_interface name="position">
                   <param name="initial_value">${initial_positions['wrist_3_joint']}</param>
                 </state_interface>
                 <state_interface name="velocity"/>
+                <state_interface name="effort"/>
             </joint>
             <joint name="robotiq_85_left_knuckle_joint">
                 <command_interface name="position"/>
+                <command_interface name="velocity"/>
+                <command_interface name="effort"/>
                 <state_interface name="position">
                   <param name="initial_value">${initial_positions['robotiq_85_left_knuckle_joint']}</param>
                 </state_interface>
                 <state_interface name="velocity"/>
+                <state_interface name="effort"/>
+            </joint>
+            <joint name="robotiq_85_right_knuckle_joint">
+                <command_interface name="position"/>
+                <command_interface name="velocity"/>
+                <command_interface name="effort"/>
+                <state_interface name="position">
+                  <param name="initial_value">${initial_positions['robotiq_85_right_knuckle_joint']}</param>
+                </state_interface>
+                <state_interface name="velocity"/>
+                <state_interface name="effort"/>
             </joint>
         </ros2_control>

File: ur5_moveit_config/srdf/ur.urdf.xacro (robot description, xacro)
@@ -3,5 +3,5 @@
     <xacro:arg name="initial_positions_file" default="initial_positions.yaml" />
     <!-- Import ur urdf file -->
-    <xacro:include filename="$(find ur_simulation_gz)/urdf/ur_gz_stand.urdf" />
+    <xacro:include filename="$(find ur_simulation_gz)/urdf/ur_gz.urdf.xacro" />
     <!-- Import control_xacro -->
     <xacro:include filename="ur.ros2_control.xacro" />
