Commit message: Tuned controllers and tested picknplace

File: robotiq/robotiq_description/urdf/robotiq_2f_85_macro.urdf.xacro (robot description, xacro)
@@ -160,47 +160,12 @@
                     <friction>
                     <ode>
-                        <mu1>10000</mu1>
-                        <mu2>10000</mu2>
+                        <mu1>100000.0</mu1>
+                        <mu2>100000.0</mu2>
                     </ode>
                     </friction>
                     <contact>
                     <ode>
-                        <kp>10000</kp>
-                        <kd>0.1</kd>
-                        <soft_cfm>0</soft_cfm>
-                        <soft_erp>0.2</soft_erp>
-                        <minDepth>0.02</minDepth>
-                        <maxVel>0.5</maxVel>
-                    </ode>
-                    </contact>
-                </surface>
-            </collision>
-            <inertial>
-                <origin xyz="-0.01456706 -0.0008 0.01649701" rpy="0 0 0" />
-                <mass value="4.268588744e-02" />
-                <inertia ixx="1.048152e-05" iyy="1.197888e-05" izz="4.22784e-06" ixy="0.0" ixz="3.5232e-6" iyz="0.0" />
-            </inertial>
-        </link>
-        <link name="${prefix}robotiq_85_right_finger_tip_link">
-            <visual>
-                <geometry>
-                    <mesh filename="file://$(find robotiq_description)/meshes/visual/2f_85/right_finger_tip.dae" />
-                </geometry>
-            </visual>
-            <collision>
-                <geometry>
-                    <mesh filename="file://$(find robotiq_description)/meshes/collision/2f_85/right_finger_tip.stl" />
-                </geometry>
-                <surface>
-                    <friction>
-                    <ode>
-                        <mu1>10000</mu1>
-                        <mu2>10000</mu2>
-                    </ode>
-                    </friction>
-                    <contact>
-                    <ode>
-                        <kp>10000</kp>
-                        <kd>0.1</kd>
+                        <kp>1e+5</kp>
+                        <kd>1</kd>
                         <soft_cfm>0</soft_cfm>
                         <soft_erp>0.2</soft_erp>
@@ -212,4 +177,39 @@
             </collision>
             <inertial>
+                <origin xyz="-0.01456706 -0.0008 0.01649701" rpy="0 0 0" />
+                <mass value="4.268588744e-02" />
+                <inertia ixx="1.048152e-05" iyy="1.197888e-05" izz="4.22784e-06" ixy="0.0" ixz="3.5232e-6" iyz="0.0" />
+            </inertial>
+        </link>
+        <link name="${prefix}robotiq_85_right_finger_tip_link">
+            <visual>
+                <geometry>
+                    <mesh filename="file://$(find robotiq_description)/meshes/visual/2f_85/right_finger_tip.dae" />
+                </geometry>
+            </visual>
+            <collision>
+                <geometry>
+                    <mesh filename="file://$(find robotiq_description)/meshes/collision/2f_85/right_finger_tip.stl" />
+                </geometry>
+                <surface>
+                    <friction>
+                    <ode>
+                        <mu1>100000.0</mu1>
+                        <mu2>100000.0</mu2>
+                    </ode>
+                    </friction>
+                    <contact>
+                    <ode>
+                        <kp>1e+5</kp>
+                        <kd>1</kd>
+                        <soft_cfm>0</soft_cfm>
+                        <soft_erp>0.2</soft_erp>
+                        <minDepth>0.002</minDepth>
+                        <maxVel>0.5</maxVel>
+                    </ode>
+                    </contact>
+                </surface>
+            </collision>
+            <inertial>
                 <origin xyz="0.01456706 5e-05 0.01649701" rpy="0 0 0" />
                 <mass value="4.268588744e-02" />
@@ -227,5 +227,5 @@
             <axis xyz="0 -1 0" />
             <origin xyz="0.03060114 0.0 0.05490452" rpy="0 0 0" />
-            <limit lower="0.0" upper="0.8" velocity="1.0" effort="28" />
+            <limit lower="0.0" upper="0.8" velocity="1.0" effort="75" />
         </joint>
         <joint name="${prefix}robotiq_85_right_knuckle_joint" type="revolute">
@@ -234,5 +234,5 @@
             <axis xyz="0 -1 0" />
             <origin xyz="-0.03060114 0.0 0.05490452" rpy="0 0 0" />
-            <limit lower="-0.8" upper="0.0" velocity="1.0" effort="28" />
+            <limit lower="-0.8" upper="0.0" velocity="1.0" effort="75" />
         </joint>
         <joint name="${prefix}robotiq_85_left_finger_joint" type="fixed">
