Commit message: Modified worlds

File: models/urdf/bottle_v2/mobility.urdf (robot description, URDF)
Before this commit: robot partnet_77699e08e3824eab47765668cf4023ed, 3 links, 2 joints
Links:
- removed link link_1
- removed link link_1_helper
- link link_0: mass 0.03 -> 5.0; geometry collision cylinder length=0.166 radius=0.04; visual mesh filename=/home/rohan/Projects/pick_n_place/src/models/urdf/bottle_v2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 scale=0.1 0.1 0.1
Joints:
- removed joint joint_1
- removed joint joint_2

File: robotiq/robotiq_description/urdf/robotiq_2f_85_macro.urdf.xacro (robot description, xacro)
@@ -157,22 +157,4 @@
                     <mesh filename="file://$(find robotiq_description)/meshes/collision/2f_85/left_finger_tip.stl" />
                 </geometry>
-                <surface>
-                    <friction>
-                    <ode>
-                        <mu1>100000.0</mu1>
-                        <mu2>100000.0</mu2>
-                    </ode>
-                    </friction>
-                    <contact>
-                    <ode>
-                        <kp>1e+5</kp>
-                        <kd>1</kd>
-                        <soft_cfm>0</soft_cfm>
-                        <soft_erp>0.2</soft_erp>
-                        <minDepth>0.002</minDepth>
-                        <maxVel>0.5</maxVel>
-                    </ode>
-                    </contact>
-                </surface>
             </collision>
             <inertial>
@@ -182,4 +164,20 @@
             </inertial>
         </link>
+        <gazebo reference="${prefix}robotiq_85_left_finger_tip_link">
+            <mu1>1000</mu1>
+            <mu2>1000</mu2>
+            <kp>1000000.0</kp>
+            <kd>100000.0</kd>
+            <slip1>0</slip1>
+            <slip2>0</slip2>
+            <minDepth>0.001</minDepth>
+            <maxVel>0</maxVel>
+            <torsional>
+                <ode>
+                    <coefficient>1000</coefficient>
+                    <slip>0</slip>
+                </ode>
+            </torsional>
+        </gazebo>
         <link name="${prefix}robotiq_85_right_finger_tip_link">
             <visual>
@@ -192,22 +190,4 @@
                     <mesh filename="file://$(find robotiq_description)/meshes/collision/2f_85/right_finger_tip.stl" />
                 </geometry>
-                <surface>
-                    <friction>
-                    <ode>
-                        <mu1>100000.0</mu1>
-                        <mu2>100000.0</mu2>
-                    </ode>
-                    </friction>
-                    <contact>
-                    <ode>
-                        <kp>1e+5</kp>
-                        <kd>1</kd>
-                        <soft_cfm>0</soft_cfm>
-                        <soft_erp>0.2</soft_erp>
-                        <minDepth>0.002</minDepth>
-                        <maxVel>0.5</maxVel>
-                    </ode>
-                    </contact>
-                </surface>
             </collision>
             <inertial>
@@ -217,4 +197,20 @@
             </inertial>
         </link>
+        <gazebo reference="${prefix}robotiq_85_right_finger_tip_link">
+            <mu1>1000</mu1>
+            <mu2>1000</mu2>
+            <kp>1000000.0</kp>
+            <kd>100000.0</kd>
+            <slip1>0</slip1>
+            <slip2>0</slip2>
+            <minDepth>0.001</minDepth>
+            <maxVel>0</maxVel>
+            <torsional>
+                <ode>
+                    <coefficient>1000</coefficient>
+                    <slip>0</slip>
+                </ode>
+            </torsional>
+        </gazebo>
         <joint name="${prefix}robotiq_85_base_joint" type="fixed">
             <parent link="${parent}" />
@@ -227,5 +223,6 @@
             <axis xyz="0 -1 0" />
             <origin xyz="0.03060114 0.0 0.05490452" rpy="0 0 0" />
-            <limit lower="0.0" upper="0.8" velocity="1.0" effort="75" />
+            <limit lower="0.0" upper="0.8" velocity="1.5" effort="500" />
+            <dynamics damping="3.0" friction="0.4"/>
         </joint>
         <joint name="${prefix}robotiq_85_right_knuckle_joint" type="revolute">
@@ -234,5 +231,6 @@
             <axis xyz="0 -1 0" />
             <origin xyz="-0.03060114 0.0 0.05490452" rpy="0 0 0" />
-            <limit lower="-0.8" upper="0.0" velocity="1.0" effort="75" />
+            <limit lower="-0.8" upper="0.0" velocity="1.5" effort="500" />
+            <dynamics damping="3.0" friction="0.4"/>
         </joint>
         <joint name="${prefix}robotiq_85_left_finger_joint" type="fixed">
